File: pead_detector_interface.kicad_sch (KiCad schematic)
At the start: 7 parts

Commit message: Changes in BOM. Add JLCpcb Part Nr
Parts:
- C600, C601: footprint (none) -> Capacitor_SMD:C_0805_2012Metric_Pad1.18x1.45mm_HandSolder; JLCBasicPart (none) -> Basic; JLCPartNr (none) -> C1710; JLCType (none) -> CL21B103KBANNNC; OriginalType (none) -> GRM216R71H103KA01D
- R600: footprint (none) -> Resistor_SMD:R_0805_2012Metric_Pad1.20x1.40mm_HandSolder; JLCBasicPart (none) -> Basic; JLCPartNr (none) -> C17414; JLCType (none) -> 0805W8F1002T5E; OriginalType (none) -> WR08X1002FTL
- R601: footprint (none) -> Resistor_SMD:R_0805_2012Metric_Pad1.20x1.40mm_HandSolder; JLCBasicPart (none) -> Basic; JLCPartNr (none) -> C17513; JLCType (none) -> 0805W8F1001T5E; OriginalType (none) -> AR05FTDW1001
Changed lines of the file:
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@@
   (symbol (lib_id "power:+5V") (at 152.4 80.01 0) (unit 1)
     (in_bom yes) (on_board yes)
-    (property "Reference" "#PWR?" (id 0) (at 152.4 83.82 0)
+    (property "Reference" "#PWR0170" (id 0) (at 152.4 83.82 0)
       (effects (font (size 1.27 1.27)) hide)
     )
@@
   (symbol (lib_id "power:VCC") (at 160.02 80.01 0) (unit 1)
     (in_bom yes) (on_board yes)
-    (property "Reference" "#PWR?" (id 0) (at 160.02 83.82 0)
+    (property "Reference" "#PWR0171" (id 0) (at 160.02 83.82 0)
       (effects (font (size 1.27 1.27)) hide)
     )
@@
   (symbol (lib_id "power:GND") (at 91.44 80.01 0) (unit 1)
     (in_bom yes) (on_board yes)
-    (property "Reference" "#PWR?" (id 0) (at 91.44 86.36 0)
+    (property "Reference" "#PWR0172" (id 0) (at 91.44 86.36 0)
       (effects (font (size 1.27 1.27)) hide)
     )
@@
   (symbol (lib_id "power:GND") (at 111.76 57.15 0) (unit 1)
     (in_bom yes) (on_board yes)
-    (property "Reference" "#PWR?" (id 0) (at 111.76 63.5 0)
+    (property "Reference" "#PWR0169" (id 0) (at 111.76 63.5 0)
       (effects (font (size 1.27 1.27)) hide)
     )
@@
   (symbol (lib_id "power:GND") (at 162.56 58.42 0) (unit 1)
     (in_bom yes) (on_board yes)
-    (property "Reference" "#PWR?" (id 0) (at 162.56 64.77 0)
+    (property "Reference" "#PWR0168" (id 0) (at 162.56 64.77 0)
       (effects (font (size 1.27 1.27)) hide)
     )
@@
   (symbol (lib_id "power:GND") (at 182.88 81.28 0) (unit 1)
     (in_bom yes) (on_board yes)
-    (property "Reference" "#PWR?" (id 0) (at 182.88 87.63 0)
+    (property "Reference" "#PWR0173" (id 0) (at 182.88 87.63 0)
       (effects (font (size 1.27 1.27)) hide)
     )
@@
       (effects (font (size 1.27 1.27)) (justify left))
     )
-    (property "Footprint" "" (id 2) (at 89.662 73.66 90)
+    (property "Footprint" "Resistor_SMD:R_0805_2012Metric_Pad1.20x1.40mm_HandSolder" (id 2) (at 89.662 73.66 90)
       (effects (font (size 1.27 1.27)) hide)
     )
     (property "Datasheet" "~" (id 3) (at 91.44 73.66 0)
+      (effects (font (size 1.27 1.27)) hide)
+    )
+    (property "JLCBasicPart" "Basic" (id 4) (at 91.44 73.66 0)
+      (effects (font (size 1.27 1.27)) hide)
+    )
+    (property "JLCPartNr" "C17414" (id 5) (at 91.44 73.66 0)
+      (effects (font (size 1.27 1.27)) hide)
+    )
+    (property "JLCType" "0805W8F1002T5E" (id 6) (at 91.44 73.66 0)
+      (effects (font (size 1.27 1.27)) hide)
+    )
+    (property "OriginalType" "WR08X1002FTL" (id 7) (at 91.44 73.66 0)
       (effects (font (size 1.27 1.27)) hide)
     )
@@
     (property "Reference" "R601" (id 0) (at 175.26 63.3538 90))
     (property "Value" "1k" (id 1) (at 175.26 65.6525 90))
-    (property "Footprint" "" (id 2) (at 175.26 70.358 90)
+    (property "Footprint" "Resistor_SMD:R_0805_2012Metric_Pad1.20x1.40mm_HandSolder" (id 2) (at 175.26 70.358 90)
       (effects (font (size 1.27 1.27)) hide)
     )
     (property "Datasheet" "~" (id 3) (at 175.26 68.58 0)
+      (effects (font (size 1.27 1.27)) hide)
+    )
+    (property "JLCBasicPart" "Basic" (id 4) (at 175.26 68.58 0)
+      (effects (font (size 1.27 1.27)) hide)
+    )
+    (property "JLCPartNr" "C17513" (id 5) (at 175.26 68.58 0)
+      (effects (font (size 1.27 1.27)) hide)
+    )
+    (property "JLCType" "0805W8F1001T5E" (id 6) (at 175.26 68.58 0)
+      (effects (font (size 1.27 1.27)) hide)
+    )
+    (property "OriginalType" "AR05FTDW1001 " (id 7) (at 175.26 68.58 0)
       (effects (font (size 1.27 1.27)) hide)
     )
@@
     (property "Reference" "C600" (id 0) (at 99.06 60.9346 90))
     (property "Value" "10n" (id 1) (at 99.06 63.246 90))
-    (property "Footprint" "" (id 2) (at 95.25 68.2752 0)
+    (property "Footprint" "Capacitor_SMD:C_0805_2012Metric_Pad1.18x1.45mm_HandSolder" (id 2) (at 95.25 68.2752 0)
       (effects (font (size 1.27 1.27)) hide)
     )
@@
       (effects (font (size 1.27 1.27)) hide)
     )
+    (property "JLCBasicPart" "Basic" (id 4) (at 99.06 67.31 0)
+      (effects (font (size 1.27 1.27)) hide)
+    )
+    (property "JLCPartNr" "C1710" (id 5) (at 99.06 67.31 0)
+      (effects (font (size 1.27 1.27)) hide)
+    )
+    (property "JLCType" "CL21B103KBANNNC" (id 6) (at 99.06 67.31 0)
+      (effects (font (size 1.27 1.27)) hide)
+    )
+    (property "OriginalType" "GRM216R71H103KA01D " (id 7) (at 99.06 67.31 0)
+      (effects (font (size 1.27 1.27)) hide)
+    )
     (pin "1")
     (pin "2")
@@
       (effects (font (size 1.27 1.27)) (justify left))
     )
-    (property "Footprint" "" (id 2) (at 183.8452 80.01 0)
+    (property "Footprint" "Capacitor_SMD:C_0805_2012Metric_Pad1.18x1.45mm_HandSolder" (id 2) (at 183.8452 80.01 0)
       (effects (font (size 1.27 1.27)) hide)
     )
@@
       (effects (font (size 1.27 1.27)) hide)
     )
+    (property "JLCBasicPart" "Basic" (id 4) (at 182.88 76.2 0)
+      (effects (font (size 1.27 1.27)) hide)
+    )
+    (property "JLCPartNr" "C1710" (id 5) (at 182.88 76.2 0)
+      (effects (font (size 1.27 1.27)) hide)
+    )
+    (property "JLCType" "CL21B103KBANNNC" (id 6) (at 182.88 76.2 0)
+      (effects (font (size 1.27 1.27)) hide)
+    )
+    (property "OriginalType" "GRM216R71H103KA01D " (id 7) (at 182.88 76.2 0)
+      (effects (font (size 1.27 1.27)) hide)
+    )

Commit message: Minor Fixes
Connections:
- net GND: now also C601.2, JP600A.1 (Pin_1)
Changed lines of the file:
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@@
+    (stroke (width 0) (type solid) (color 0 0 0 0))
+  )
+  (wire (pts (xy 111.76 55.88) (xy 111.76 57.15))
     (stroke (width 0) (type solid) (color 0 0 0 0))
   )
@@
     (stroke (width 0) (type solid) (color 0 0 0 0))
   )
+  (wire (pts (xy 182.88 80.01) (xy 182.88 81.28))
+    (stroke (width 0) (type solid) (color 0 0 0 0))
+  )

Commit message: working on BOM. Small Fixes in Schematics
Parts:
- renumbered JP600A to JP601, JP600B to JP602
Changed lines of the file:
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@@
   (symbol (lib_id "Connector_Generic:Conn_01x03") (at 114.3 50.8 90) (unit 1)
     (in_bom yes) (on_board yes)
-    (property "Reference" "JP600A" (id 0) (at 118.9736 51.689 90)
+    (property "Reference" "JP601" (id 0) (at 118.9736 51.689 90)
       (effects (font (size 1.27 1.27)) (justify right))
     )
@@
   (symbol (lib_id "Connector_Generic:Conn_01x05") (at 157.48 50.8 90) (unit 1)
     (in_bom yes) (on_board yes)
-    (property "Reference" "JP600B" (id 0) (at 164.6936 51.689 90)
+    (property "Reference" "JP602" (id 0) (at 164.6936 51.689 90)
       (effects (font (size 1.27 1.27)) (justify right))
     )

Commit message: Footprints assigned. Testpoints added
Parts:
- JP601: footprint (none) -> Connector_PinHeader_2.54mm:PinHeader_1x03_P2.54mm_Vertical
- JP602: footprint (none) -> Connector_PinHeader_2.54mm:PinHeader_1x05_P2.54mm_Vertical
- TP17: footprint (none) -> TestPoint:TestPoint_THTPad_1.5x1.5mm_Drill0.7mm
Changed lines of the file:
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@@
       (effects (font (size 1.27 1.27)) (justify left))
     )
-    (property "Footprint" "" (id 2) (at 187.96 63.5 0)
+    (property "Footprint" "TestPoint:TestPoint_THTPad_1.5x1.5mm_Drill0.7mm" (id 2) (at 187.96 63.5 0)
       (effects (font (size 1.27 1.27)) hide)
     )
@@
       (effects (font (size 1.27 1.27)) (justify right))
     )
-    (property "Footprint" "" (id 2) (at 114.3 50.8 0)
+    (property "Footprint" "Connector_PinHeader_2.54mm:PinHeader_1x03_P2.54mm_Vertical" (id 2) (at 114.3 50.8 0)
       (effects (font (size 1.27 1.27)) hide)
     )
@@
       (effects (font (size 1.27 1.27)) (justify right))
     )
-    (property "Footprint" "" (id 2) (at 157.48 50.8 0)
-      (effects (font (size 1.27 1.27)) hide)
-    )
+    (property "Footprint" "Connector_PinHeader_2.54mm:PinHeader_1x05_P2.54mm_Vertical" (id 2) (at 157.48 50.8 0)
+      (effects (font (size 1.27 1.27)) hide)
+    )

Commit message: Started PCB. Placed Parts
Parts:
- JP601: footprint Connector_PinHeader_2.54mm:PinHeader_1x03_P2.54mm_Vertical -> Connector_PinSocket_2.54mm:PinSocket_1x03_P2.54mm_Vertical
- JP602: footprint Connector_PinHeader_2.54mm:PinHeader_1x05_P2.54mm_Vertical -> Connector_PinSocket_2.54mm:PinSocket_1x05_P2.54mm_Vertical
Changed lines of the file:
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@@
       (effects (font (size 1.27 1.27)) (justify right))
     )
-    (property "Footprint" "Connector_PinHeader_2.54mm:PinHeader_1x03_P2.54mm_Vertical" (id 2) (at 114.3 50.8 0)
+    (property "Footprint" "Connector_PinSocket_2.54mm:PinSocket_1x03_P2.54mm_Vertical" (id 2) (at 114.3 50.8 0)
       (effects (font (size 1.27 1.27)) hide)
     )
@@
       (effects (font (size 1.27 1.27)) (justify right))
     )
-    (property "Footprint" "Connector_PinHeader_2.54mm:PinHeader_1x05_P2.54mm_Vertical" (id 2) (at 157.48 50.8 0)
+    (property "Footprint" "Connector_PinSocket_2.54mm:PinSocket_1x05_P2.54mm_Vertical" (id 2) (at 157.48 50.8 0)
       (effects (font (size 1.27 1.27)) hide)
     )

Commit message: Removed optionals parts. Cleaned up Schematics
Parts:
- added JP600, JP603, JP604, JP605: SolderJumper_2_Bridged, Jumper:SolderJumper-2_P1.3mm_Bridged_Pad1.0x1.5mm, symbol Jumper:SolderJumper_2_Bridged
Connections:
- net DISCR1.1_TERM: now also JP603.1 (A); no longer JP601.3 (Pin_3)
- net ENERGY1: now also JP605.2 (B); no longer C601.1, R601.2, TP17.1
- net HI_GAIN: now also JP604.1 (A); no longer JP602.1 (Pin_1)
- net INP1_BUFFER: now also JP600.1 (A); no longer C600.2, R600.1
- new net: C601.1, JP605.1 (A), R601.2, TP17.1
- new net: C600.2, JP600.2 (B), R600.1
- new net: JP601.3 (Pin_3), JP603.2 (B)
- new net: JP602.1 (Pin_1), JP604.2 (B)
Changed lines of the file:
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@@
   (junction (at 91.44 67.31) (diameter 1.016) (color 0 0 0 0))
   (junction (at 182.88 68.58) (diameter 1.016) (color 0 0 0 0))
+  (wire (pts (xy 73.66 67.31) (xy 77.47 67.31))
+    (stroke (width 0) (type solid) (color 0 0 0 0))
+  )
   (wire (pts (xy 85.09 67.31) (xy 91.44 67.31))
     (stroke (width 0) (type solid) (color 0 0 0 0))
@@
     (stroke (width 0) (type solid) (color 0 0 0 0))
   )
-  (wire (pts (xy 116.84 55.88) (xy 116.84 62.23))
-    (stroke (width 0) (type solid) (color 0 0 0 0))
-  )
-  (wire (pts (xy 152.4 55.88) (xy 152.4 62.23))
+  (wire (pts (xy 116.84 55.88) (xy 116.84 57.15))
+    (stroke (width 0) (type solid) (color 0 0 0 0))
+  )
+  (wire (pts (xy 116.84 64.77) (xy 116.84 67.31))
+    (stroke (width 0) (type solid) (color 0 0 0 0))
+  )
+  (wire (pts (xy 152.4 55.88) (xy 152.4 57.15))
     (stroke (width 0) (type solid) (color 0 0 0 0))
   )
@@
     (stroke (width 0) (type solid) (color 0 0 0 0))
   )
-  (global_label "INP1_BUFFER" (shape input) (at 85.09 67.31 180)
+  (wire (pts (xy 195.58 68.58) (xy 196.85 68.58))
+    (stroke (width 0) (type solid) (color 0 0 0 0))
+  )
+  (global_label "INP1_BUFFER" (shape input) (at 73.66 67.31 180)
     (effects (font (size 1.27 1.27)) (justify right))
-    (property "Intersheet References" "${INTERSHEET_REFS}" (id 0) (at 68.5739 67.2306 0)
+    (property "Intersheet References" "${INTERSHEET_REFS}" (id 0) (at 57.1439 67.2306 0)
       (effects (font (size 1.27 1.27)) (justify right) hide)
     )
   )
-  (global_label "DISCR1.1_TERM" (shape input) (at 116.84 62.23 270)
+  (global_label "DISCR1.1_TERM" (shape input) (at 116.84 67.31 270)
     (effects (font (size 1.27 1.27)) (justify right))
-    (property "Intersheet References" "${INTERSHEET_REFS}" (id 0) (at 116.7606 80.6209 90)
+    (property "Intersheet References" "${INTERSHEET_REFS}" (id 0) (at 116.7606 85.7009 90)
       (effects (font (size 1.27 1.27)) (justify right) hide)
     )
   )
-  (global_label "HI_GAIN" (shape input) (at 152.4 62.23 270)
+  (global_label "HI_GAIN" (shape input) (at 152.4 64.77 270)
     (effects (font (size 1.27 1.27)) (justify right))
-    (property "Intersheet References" "${INTERSHEET_REFS}" (id 0) (at 152.3206 73.3638 90)
+    (property "Intersheet References" "${INTERSHEET_REFS}" (id 0) (at 152.3206 75.9038 90)
       (effects (font (size 1.27 1.27)) (justify right) hide)
     )
   )
-  (global_label "ENERGY1" (shape input) (at 187.96 68.58 0)
+  (global_label "ENERGY1" (shape input) (at 196.85 68.58 0)
     (effects (font (size 1.27 1.27)) (justify left))
-    (property "Intersheet References" "${INTERSHEET_REFS}" (id 0) (at 200.3638 68.5006 0)
+    (property "Intersheet References" "${INTERSHEET_REFS}" (id 0) (at 209.2538 68.5006 0)
       (effects (font (size 1.27 1.27)) (justify left) hide)
     )
@@
     (pin "1")
   )
+  (symbol (lib_id "Jumper:SolderJumper_2_Bridged") (at 81.28 67.31 0) (unit 1)
+    (in_bom no) (on_board yes)
+    (property "Reference" "JP600" (id 0) (at 81.28 64.2578 0))
+    (property "Value" "SolderJumper_2_Bridged" (id 1) (at 81.28 65.2865 0)
+      (effects (font (size 1.27 1.27)) hide)
+    )
+    (property "Footprint" "Jumper:SolderJumper-2_P1.3mm_Bridged_Pad1.0x1.5mm" (id 2) (at 81.28 67.31 0)
+      (effects (font (size 1.27 1.27)) hide)
+    )
+    (property "Datasheet" "~" (id 3) (at 81.28 67.31 0)
+      (effects (font (size 1.27 1.27)) hide)
+    )
+    (pin "1")
+    (pin "2")
+  )
+  (symbol (lib_id "Jumper:SolderJumper_2_Bridged") (at 116.84 60.96 90) (unit 1)
+    (in_bom no) (on_board yes)
+    (property "Reference" "JP603" (id 0) (at 120.1378 60.96 0))
+    (property "Value" "SolderJumper_2_Bridged" (id 1) (at 114.8165 60.96 0)
+      (effects (font (size 1.27 1.27)) hide)
+    )
+    (property "Footprint" "Jumper:SolderJumper-2_P1.3mm_Bridged_Pad1.0x1.5mm" (id 2) (at 116.84 60.96 0)
+      (effects (font (size 1.27 1.27)) hide)
+    )
+    (property "Datasheet" "~" (id 3) (at 116.84 60.96 0)
+      (effects (font (size 1.27 1.27)) hide)
+    )
+    (pin "1")
+    (pin "2")
+  )
+  (symbol (lib_id "Jumper:SolderJumper_2_Bridged") (at 152.4 60.96 90) (unit 1)
+    (in_bom no) (on_board yes)
+    (property "Reference" "JP604" (id 0) (at 149.3478 60.96 0))
+    (property "Value" "SolderJumper_2_Bridged" (id 1) (at 150.3765 60.96 0)
+      (effects (font (size 1.27 1.27)) hide)
+    )
+    (property "Footprint" "Jumper:SolderJumper-2_P1.3mm_Bridged_Pad1.0x1.5mm" (id 2) (at 152.4 60.96 0)
+      (effects (font (size 1.27 1.27)) hide)
+    )
+    (property "Datasheet" "~" (id 3) (at 152.4 60.96 0)
+      (effects (font (size 1.27 1.27)) hide)
+    )
+    (pin "1")
+    (pin "2")
+  )
+  (symbol (lib_id "Jumper:SolderJumper_2_Bridged") (at 191.77 68.58 0) (unit 1)
+    (in_bom no) (on_board yes)
+    (property "Reference" "JP605" (id 0) (at 191.77 65.5278 0))
+    (property "Value" "SolderJumper_2_Bridged" (id 1) (at 191.77 66.5565 0)
+      (effects (font (size 1.27 1.27)) hide)
+    )
+    (property "Footprint" "Jumper:SolderJumper-2_P1.3mm_Bridged_Pad1.0x1.5mm" (id 2) (at 191.77 68.58 0)
+      (effects (font (size 1.27 1.27)) hide)
+    )
+    (property "Datasheet" "~" (id 3) (at 191.77 68.58 0)
+      (effects (font (size 1.27 1.27)) hide)
+    )
+    (pin "1")
+    (pin "2")
+  )
   (symbol (lib_id "Device:R") (at 91.44 73.66 0) (unit 1)
