File: cdu-lite.kicad_sch (KiCad schematic)
At the start: 0 parts

Commit message: Silkscreen edided. Minor improvements
Other:
- sheet Pead Detector Interface renamed Peak Detector Interface
- sheet Peak Detector Interface: file pead_detector_interface.kicad_sch -> peak_detector_interface.kicad_sch
Changed lines of the file:
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@@
     (stroke (width 0) (type solid) (color 132 0 132 1))
     (fill (color 255 255 255 0.0000))
-    (property "Sheet name" "Pead Detector Interface" (id 0) (at 215.9 27.3045 0)
+    (property "Sheet name" "Peak Detector Interface" (id 0) (at 215.9 27.3045 0)
       (effects (font (size 1.27 1.27)) (justify left bottom))
     )
-    (property "Sheet file" "pead_detector_interface.kicad_sch" (id 1) (at 215.9 51.3085 0)
+    (property "Sheet file" "peak_detector_interface.kicad_sch" (id 1) (at 215.9 51.3085 0)
       (effects (font (size 1.27 1.27)) (justify left top))
     )
