File: digital_pulseprocessor.kicad_sch (KiCad schematic)
At the start: 17 parts, among them J300 SolderJumper_2_Open, J310 Conn_02x03_Odd_Even, U300 SN74LV221AD, U301 SN74LV221AD

Commit message: Refactored schematic to better show relationship in main schematic
Parts:
- removed J310: Conn_02x03_Odd_Even, Connector_PinHeader_2.54mm:PinHeader_2x03_P2.54mm_Vertical, symbol Connector_Generic:Conn_02x03_Odd_Even

Commit message: Cleaned up board, replaced GPIO footprint with unshrouded version
Connections:
- net VCC renamed 3V3
Changed lines of the file:
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@@
     )
   )
-  (hierarchical_label "VCC" (shape input) (at 41.91 64.77 180)
+  (hierarchical_label "3V3" (shape input) (at 41.91 64.77 180)
     (effects (font (size 1.27 1.27)) (justify right))
   )
-  (hierarchical_label "VCC" (shape input) (at 44.45 151.13 90)
+  (hierarchical_label "3V3" (shape input) (at 41.91 124.46 180)
+    (effects (font (size 1.27 1.27)) (justify right))
+  )
+  (hierarchical_label "3V3" (shape input) (at 44.45 151.13 90)
     (effects (font (size 1.27 1.27)) (justify left))
   )
@@
     (effects (font (size 1.27 1.27)) (justify right))
   )
-  (hierarchical_label "VCC" (shape input) (at 58.42 25.4 90)
+  (hierarchical_label "3V3" (shape input) (at 58.42 25.4 90)
     (effects (font (size 1.27 1.27)) (justify left))
   )
-  (hierarchical_label "VCC" (shape input) (at 58.42 85.09 90)
+  (hierarchical_label "3V3" (shape input) (at 58.42 85.09 90)
     (effects (font (size 1.27 1.27)) (justify left))
   )
@@
     (effects (font (size 1.27 1.27)) (justify left))
   )
-  (hierarchical_label "VCC" (shape input) (at 93.98 151.13 90)
+  (hierarchical_label "3V3" (shape input) (at 93.98 151.13 90)
     (effects (font (size 1.27 1.27)) (justify left))
   )
@@
     (effects (font (size 1.27 1.27)) (justify left))
   )
-  (hierarchical_label "VCC" (shape input) (at 207.645 93.98 180)
+  (hierarchical_label "3V3" (shape input) (at 207.645 93.98 180)
     (effects (font (size 1.27 1.27)) (justify right))
   )
-  (hierarchical_label "VCC" (shape input) (at 209.55 54.61 90)
+  (hierarchical_label "3V3" (shape input) (at 209.55 54.61 90)
     (effects (font (size 1.27 1.27)) (justify left))
   )
@@
     (effects (font (size 1.27 1.27)) (justify left))
   )
-  (symbol (lib_id "power:VCC") (at 41.91 124.46 0) (unit 1)
-    (in_bom yes) (on_board yes)
-    (property "Reference" "#PWR0163" (id 0) (at 41.91 128.27 0)
-      (effects (font (size 1.27 1.27)) hide)
-    )
-    (property "Value" "VCC" (id 1) (at 42.2783 120.1356 0))
-    (property "Footprint" "" (id 2) (at 41.91 124.46 0)
-      (effects (font (size 1.27 1.27)) hide)
-    )
-    (property "Datasheet" "" (id 3) (at 41.91 124.46 0)
-      (effects (font (size 1.27 1.27)) hide)
-    )
-    (pin "1")
-  )
   (symbol (lib_id "Connector:TestPoint") (at 121.92 71.12 270) (unit 1)
