File: digital_pulseprocessor.kicad_sch (KiCad schematic)
At the start: 17 parts, among them J300 SolderJumper_2_Open, J310 Conn_02x03_Odd_Even, U300 SN74LV221AD, U301 SN74LV221AD

Commit message: some changes after first test of boards. Package of SN74LV221AD changed to SOIC-16.
Parts:
- C300: JLCplace (none) -> C1814; Supplier (none) -> LCSC; alternativ supply (none) -> mouser; alternativ supply part nr. (none) -> CC0805JRNPO9BN330
- C303: JLCplace (none) -> C46653; Supplier (none) -> LCSC
- C304, C564, C566: JLCplace (none) -> C49678; Supplier (none) -> LCSC
- J300, TP26, TP27, TP28: Supplier (none) -> --
- J310: OriginalType (none) -> 649-1012938190601BLF; Supplier (none) -> Mouser
- R300, R303: JLCplace (none) -> C17513; Supplier (none) -> LCSC
- R304: JLCplace (none) -> C17709; Supplier (none) -> LCSC
- R306, R311: JLCplace (none) -> C17738; Supplier (none) -> LCSC
- U300, U301: footprint Package_SO:SOIC-16W_7.5x10.3mm_P1.27mm -> Package_SO:SOIC-16_3.9x9.9mm_P1.27mm; JLCBasicPart (none) -> Extended; JLCPartNr (none) -> C201537; JLCType (none) -> SN74LV221ADR
Changed lines of the file:
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@@
+      (effects (font (size 1.27 1.27)) hide)
+    )
+    (property "Supplier" "--" (id 4) (at 121.92 71.12 0)
       (effects (font (size 1.27 1.27)) hide)
     )
@@
       (effects (font (size 1.27 1.27)) hide)
     )
+    (property "Supplier" "--" (id 4) (at 176.53 87.63 0)
+      (effects (font (size 1.27 1.27)) hide)
+    )
     (pin "1")
   )
@@
     )
     (property "Datasheet" "~" (id 3) (at 261.62 83.82 0)
+      (effects (font (size 1.27 1.27)) hide)
+    )
+    (property "Supplier" "--" (id 4) (at 256.54 83.82 0)
       (effects (font (size 1.27 1.27)) hide)
     )
@@
       (effects (font (size 1.27 1.27)) hide)
     )
+    (property "Supplier" "--" (id 4) (at 222.25 113.03 0)
+      (effects (font (size 1.27 1.27)) hide)
+    )
     (pin "1")
     (pin "2")
@@
       (effects (font (size 1.27 1.27)) hide)
     )
+    (property "Supplier" "LCSC" (id 8) (at 58.42 31.75 0)
+      (effects (font (size 1.27 1.27)) hide)
+    )
+    (property "JLCplace" "C17513" (id 9) (at 58.42 31.75 0)
+      (effects (font (size 1.27 1.27)) hide)
+    )
     (pin "1")
     (pin "2")
@@
       (effects (font (size 1.27 1.27)) hide)
     )
+    (property "Supplier" "LCSC" (id 8) (at 58.42 91.44 0)
+      (effects (font (size 1.27 1.27)) hide)
+    )
+    (property "JLCplace" "C17709" (id 9) (at 58.42 91.44 0)
+      (effects (font (size 1.27 1.27)) hide)
+    )
     (pin "1")
     (pin "2")
@@
       (effects (font (size 1.27 1.27)) hide)
     )
+    (property "Supplier" "LCSC" (id 8) (at 114.3 63.5 0)
+      (effects (font (size 1.27 1.27)) hide)
+    )
+    (property "JLCplace" "C17738" (id 9) (at 114.3 63.5 0)
+      (effects (font (size 1.27 1.27)) hide)
+    )
     (pin "1")
     (pin "2")
@@
       (effects (font (size 1.27 1.27)) hide)
     )
+    (property "Supplier" "LCSC" (id 8) (at 209.55 60.96 0)
+      (effects (font (size 1.27 1.27)) hide)
+    )
+    (property "JLCplace" "C17513" (id 9) (at 209.55 60.96 0)
+      (effects (font (size 1.27 1.27)) hide)
+    )
     (pin "1")
     (pin "2")
@@
       (effects (font (size 1.27 1.27)) hide)
     )
+    (property "Supplier" "LCSC" (id 8) (at 248.92 86.36 0)
+      (effects (font (size 1.27 1.27)) hide)
+    )
+    (property "JLCplace" "C17738" (id 9) (at 248.92 86.36 0)
+      (effects (font (size 1.27 1.27)) hide)
+    )
     (pin "1")
     (pin "2")
@@
       (effects (font (size 1.27 1.27)) hide)
     )
+    (property "Supplier" "LCSC" (id 8) (at 24.13 167.64 0)
+      (effects (font (size 1.27 1.27)) hide)
+    )
+    (property "JLCplace" "C49678" (id 9) (at 24.13 167.64 0)
+      (effects (font (size 1.27 1.27)) hide)
+    )
     (pin "1")
     (pin "2")
@@
       (effects (font (size 1.27 1.27)) hide)
     )
+    (property "Supplier" "LCSC" (id 8) (at 58.42 41.91 0)
+      (effects (font (size 1.27 1.27)) hide)
+    )
+    (property "JLCplace" "C1814" (id 9) (at 58.42 41.91 0)
+      (effects (font (size 1.27 1.27)) hide)
+    )
+    (property "alternativ supply" "mouser" (id 10) (at 58.42 41.91 0)
+      (effects (font (size 1.27 1.27)) hide)
+    )
+    (property "alternativ supply part nr." "CC0805JRNPO9BN330" (id 11) (at 58.42 41.91 0)
+      (effects (font (size 1.27 1.27)) hide)
+    )
     (pin "1")
     (pin "2")
@@
       (effects (font (size 1.27 1.27)) hide)
     )
+    (property "Supplier" "LCSC" (id 8) (at 58.42 101.6 0)
+      (effects (font (size 1.27 1.27)) hide)
+    )
+    (property "JLCplace" "C49678" (id 9) (at 58.42 101.6 0)
+      (effects (font (size 1.27 1.27)) hide)
+    )
     (pin "1")
     (pin "2")
@@
       (effects (font (size 1.27 1.27)) hide)
     )
+    (property "Supplier" "LCSC" (id 8) (at 76.2 167.64 0)
+      (effects (font (size 1.27 1.27)) hide)
+    )
+    (property "JLCplace" "C49678" (id 9) (at 76.2 167.64 0)
+      (effects (font (size 1.27 1.27)) hide)
+    )
     (pin "1")
     (pin "2")
@@
     )
     (property "OriginalType" "0805B102K500CT " (id 7) (at 209.55 71.12 0)
+      (effects (font (size 1.27 1.27)) hide)
+    )
+    (property "Supplier" "LCSC" (id 8) (at 209.55 71.12 0)
+      (effects (font (size 1.27 1.27)) hide)
+    )
+    (property "JLCplace" "C46653" (id 9) (at 209.55 71.12 0)
       (effects (font (size 1.27 1.27)) hide)
     )
@@
       (effects (font (size 1.27 1.27)) hide)
     )
+    (property "OriginalType" "649-1012938190601BLF" (id 4) (at 148.59 129.54 0)
+      (effects (font (size 1.27 1.27)) hide)
+    )
+    (property "Supplier" "Mouser" (id 5) (at 148.59 129.54 0)
+      (effects (font (size 1.27 1.27)) hide)
+    )
     (pin "1")
     (pin "2")
@@
     (property "Reference" "U300" (id 0) (at 34.29 155.5814 0))
     (property "Value" "SN74LV221AD" (id 1) (at 35.56 157.8801 0))
-    (property "Footprint" "Package_SO:SOIC-16W_7.5x10.3mm_P1.27mm" (id 2) (at 44.45 167.64 0)
+    (property "Footprint" "Package_SO:SOIC-16_3.9x9.9mm_P1.27mm" (id 2) (at 44.45 167.64 0)
       (effects (font (size 1.27 1.27)) hide)
     )
@@
     )
     (property "Supplier" "Mouser" (id 5) (at 44.45 167.64 0)
+      (effects (font (size 1.27 1.27)) hide)
+    )
+    (property "JLCBasicPart" "Extended" (id 6) (at 44.45 167.64 0)
+      (effects (font (size 1.27 1.27)) hide)
+    )
+    (property "JLCPartNr" "C201537" (id 7) (at 44.45 167.64 0)
+      (effects (font (size 1.27 1.27)) hide)
+    )
+    (property "JLCType" "SN74LV221ADR" (id 8) (at 44.45 167.64 0)
       (effects (font (size 1.27 1.27)) hide)
     )
@@
     (property "Reference" "U301" (id 0) (at 82.55 155.5814 0))
     (property "Value" "SN74LV221AD" (id 1) (at 85.09 157.8801 0))
-    (property "Footprint" "Package_SO:SOIC-16W_7.5x10.3mm_P1.27mm" (id 2) (at 93.98 167.64 0)
+    (property "Footprint" "Package_SO:SOIC-16_3.9x9.9mm_P1.27mm" (id 2) (at 93.98 167.64 0)
       (effects (font (size 1.27 1.27)) hide)
     )
@@
     )
     (property "Supplier" "Mouser" (id 5) (at 93.98 167.64 0)
+      (effects (font (size 1.27 1.27)) hide)
+    )
+    (property "JLCBasicPart" "Extended" (id 6) (at 93.98 167.64 0)
+      (effects (font (size 1.27 1.27)) hide)
+    )
+    (property "JLCPartNr" "C201537" (id 7) (at 93.98 167.64 0)
+      (effects (font (size 1.27 1.27)) hide)
+    )
+    (property "JLCType" "SN74LV221ADR" (id 8) (at 93.98 167.64 0)
       (effects (font (size 1.27 1.27)) hide)
     )
@@
     (property "Reference" "U300" (id 0) (at 71.12 71.7614 0))
     (property "Value" "SN74LV221AD" (id 1) (at 71.12 74.0664 0))
-    (property "Footprint" "Package_SO:SOIC-16W_7.5x10.3mm_P1.27mm" (id 2) (at 71.12 62.23 0)
+    (property "Footprint" "Package_SO:SOIC-16_3.9x9.9mm_P1.27mm" (id 2) (at 71.12 62.23 0)
       (effects (font (size 1.27 1.27)) hide)
     )
@@
     )
     (property "Supplier" "Mouser" (id 5) (at 71.12 62.23 0)
+      (effects (font (size 1.27 1.27)) hide)
+    )
+    (property "JLCBasicPart" "Extended" (id 6) (at 71.12 62.23 0)
+      (effects (font (size 1.27 1.27)) hide)
+    )
+    (property "JLCPartNr" "C201537" (id 7) (at 71.12 62.23 0)
+      (effects (font (size 1.27 1.27)) hide)
+    )
+    (property "JLCType" "SN74LV221ADR" (id 8) (at 71.12 62.23 0)
       (effects (font (size 1.27 1.27)) hide)
     )
@@
     (property "Reference" "U300" (id 0) (at 71.12 131.4514 0))
     (property "Value" "SN74LV221AD" (id 1) (at 71.12 133.7501 0))
-    (property "Footprint" "Package_SO:SOIC-16W_7.5x10.3mm_P1.27mm" (id 2) (at 71.12 121.92 0)
+    (property "Footprint" "Package_SO:SOIC-16_3.9x9.9mm_P1.27mm" (id 2) (at 71.12 121.92 0)
       (effects (font (size 1.27 1.27)) hide)
     )
@@
     )
     (property "Supplier" "Mouser" (id 5) (at 71.12 121.92 0)
+      (effects (font (size 1.27 1.27)) hide)
+    )
+    (property "JLCBasicPart" "Extended" (id 6) (at 71.12 121.92 0)
+      (effects (font (size 1.27 1.27)) hide)
+    )
+    (property "JLCPartNr" "C201537" (id 7) (at 71.12 121.92 0)
+      (effects (font (size 1.27 1.27)) hide)
+    )
+    (property "JLCType" "SN74LV221ADR" (id 8) (at 71.12 121.92 0)
       (effects (font (size 1.27 1.27)) hide)
     )
@@
     (property "Reference" "U301" (id 0) (at 222.25 100.965 0))
     (property "Value" "SN74LV221AD" (id 1) (at 222.25 103.2701 0))
-    (property "Footprint" "Package_SO:SOIC-16W_7.5x10.3mm_P1.27mm" (id 2) (at 222.25 91.44 0)
+    (property "Footprint" "Package_SO:SOIC-16_3.9x9.9mm_P1.27mm" (id 2) (at 222.25 91.44 0)
       (effects (font (size 1.27 1.27)) hide)
     )
@@
     )
     (property "Supplier" "Mouser" (id 5) (at 222.25 91.44 0)
+      (effects (font (size 1.27 1.27)) hide)
+    )
+    (property "JLCBasicPart" "Extended" (id 6) (at 222.25 91.44 0)
+      (effects (font (size 1.27 1.27)) hide)
+    )
+    (property "JLCPartNr" "C201537" (id 7) (at 222.25 91.44 0)
+      (effects (font (size 1.27 1.27)) hide)
+    )
+    (property "JLCType" "SN74LV221ADR" (id 8) (at 222.25 91.44 0)
       (effects (font (size 1.27 1.27)) hide)
     )
@@
     (property "Reference" "U301" (id 0) (at 228.6 153.035 0))
     (property "Value" "SN74LV221AD" (id 1) (at 228.6 155.3401 0))
-    (property "Footprint" "Package_SO:SOIC-16W_7.5x10.3mm_P1.27mm" (id 2) (at 228.6 143.51 0)
+    (property "Footprint" "Package_SO:SOIC-16_3.9x9.9mm_P1.27mm" (id 2) (at 228.6 143.51 0)
       (effects (font (size 1.27 1.27)) hide)
     )
@@
       (effects (font (size 1.27 1.27)) hide)
     )
+    (property "JLCBasicPart" "Extended" (id 6) (at 228.6 143.51 0)
+      (effects (font (size 1.27 1.27)) hide)
+    )
+    (property "JLCPartNr" "C201537" (id 7) (at 228.6 143.51 0)
+      (effects (font (size 1.27 1.27)) hide)
+    )
+    (property "JLCType" "SN74LV221ADR" (id 8) (at 228.6 143.51 0)
+      (effects (font (size 1.27 1.27)) hide)
+    )
