File: peak_detector_interface.kicad_sch (KiCad schematic)
At the start: 11 parts

Commit message: Refactored schematic to better show relationship in main schematic
Changed lines of the file:
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@@
-(kicad_sch (version 20210406) (generator eeschema)
+(kicad_sch (version 20210621) (generator eeschema)
   (paper "A4")
   (junction (at 91.44 67.31) (diameter 1.016) (color 0 0 0 0))
@@
     (stroke (width 0) (type solid) (color 0 0 0 0))
   )
-  (wire (pts (xy 152.4 82.55) (xy 152.4 80.01))
-    (stroke (width 0) (type solid) (color 0 0 0 0))
-  )
   (wire (pts (xy 154.94 55.88) (xy 154.94 82.55))
     (stroke (width 0) (type solid) (color 0 0 0 0))
   )
-  (wire (pts (xy 154.94 82.55) (xy 152.4 82.55))
-    (stroke (width 0) (type solid) (color 0 0 0 0))
-  )
   (wire (pts (xy 157.48 55.88) (xy 157.48 82.55))
-    (stroke (width 0) (type solid) (color 0 0 0 0))
-  )
-  (wire (pts (xy 157.48 82.55) (xy 160.02 82.55))
     (stroke (width 0) (type solid) (color 0 0 0 0))
   )
@@
   )
   (wire (pts (xy 160.02 68.58) (xy 171.45 68.58))
-    (stroke (width 0) (type solid) (color 0 0 0 0))
-  )
-  (wire (pts (xy 160.02 82.55) (xy 160.02 80.01))
     (stroke (width 0) (type solid) (color 0 0 0 0))
   )
@@
     (stroke (width 0) (type solid) (color 0 0 0 0))
   )
-  (global_label "INP1_BUFFER" (shape input) (at 73.66 67.31 180)
+  (hierarchical_label "INP1_BUFFER" (shape input) (at 73.66 67.31 180)
     (effects (font (size 1.27 1.27)) (justify right))
-    (property "Intersheet References" "${INTERSHEET_REFS}" (id 0) (at 57.1439 67.2306 0)
-      (effects (font (size 1.27 1.27)) (justify right) hide)
-    )
   )
-  (global_label "DISCR1.1_TERM" (shape input) (at 116.84 67.31 270)
+  (hierarchical_label "DISCR1.1_TERM" (shape input) (at 116.84 67.31 270)
     (effects (font (size 1.27 1.27)) (justify right))
-    (property "Intersheet References" "${INTERSHEET_REFS}" (id 0) (at 116.7606 85.7009 90)
-      (effects (font (size 1.27 1.27)) (justify right) hide)
-    )
   )
-  (global_label "HI_GAIN" (shape input) (at 152.4 64.77 270)
+  (hierarchical_label "HI_GAIN" (shape output) (at 152.4 64.77 270)
     (effects (font (size 1.27 1.27)) (justify right))
-    (property "Intersheet References" "${INTERSHEET_REFS}" (id 0) (at 152.3206 75.9038 90)
-      (effects (font (size 1.27 1.27)) (justify right) hide)
-    )
   )
-  (global_label "ENERGY1" (shape input) (at 196.85 68.58 0)
+  (hierarchical_label "+5V" (shape input) (at 154.94 82.55 270)
+    (effects (font (size 1.27 1.27)) (justify right))
+  )
+  (hierarchical_label "VCC" (shape input) (at 157.48 82.55 270)
+    (effects (font (size 1.27 1.27)) (justify right))
+  )
+  (hierarchical_label "ENERGY1" (shape output) (at 196.85 68.58 0)
     (effects (font (size 1.27 1.27)) (justify left))
-    (property "Intersheet References" "${INTERSHEET_REFS}" (id 0) (at 209.2538 68.5006 0)
-      (effects (font (size 1.27 1.27)) (justify left) hide)
-    )
-  )
-  (symbol (lib_id "power:+5V") (at 152.4 80.01 0) (unit 1)
-    (in_bom yes) (on_board yes)
-    (property "Reference" "#PWR0170" (id 0) (at 152.4 83.82 0)
-      (effects (font (size 1.27 1.27)) hide)
-    )
-    (property "Value" "+5V" (id 1) (at 152.7683 75.6856 0))
-    (property "Footprint" "" (id 2) (at 152.4 80.01 0)
-      (effects (font (size 1.27 1.27)) hide)
-    )
-    (property "Datasheet" "" (id 3) (at 152.4 80.01 0)
-      (effects (font (size 1.27 1.27)) hide)
-    )
-    (pin "1")
-  )
-  (symbol (lib_id "power:VCC") (at 160.02 80.01 0) (unit 1)
-    (in_bom yes) (on_board yes)
-    (property "Reference" "#PWR0171" (id 0) (at 160.02 83.82 0)
-      (effects (font (size 1.27 1.27)) hide)
-    )
-    (property "Value" "VCC" (id 1) (at 160.3883 75.6856 0))
-    (property "Footprint" "" (id 2) (at 160.02 80.01 0)
-      (effects (font (size 1.27 1.27)) hide)
-    )
-    (property "Datasheet" "" (id 3) (at 160.02 80.01 0)
-      (effects (font (size 1.27 1.27)) hide)
-    )
-    (pin "1")
   )
   (symbol (lib_id "Connector:TestPoint") (at 182.88 63.5 0) (unit 1)

Commit message: Cleaned up board, replaced GPIO footprint with unshrouded version
Connections:
- net +5V renamed 5V
- net VCC renamed 3V3
Changed lines of the file:
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@@
     (effects (font (size 1.27 1.27)) (justify right))
   )
-  (hierarchical_label "+5V" (shape input) (at 154.94 82.55 270)
+  (hierarchical_label "5V" (shape input) (at 154.94 82.55 270)
     (effects (font (size 1.27 1.27)) (justify right))
   )
-  (hierarchical_label "VCC" (shape input) (at 157.48 82.55 270)
+  (hierarchical_label "3V3" (shape input) (at 157.48 82.55 270)
     (effects (font (size 1.27 1.27)) (justify right))
   )
