File: peak_detector_interface.kicad_sch (KiCad schematic)
At the start: 11 parts

Commit message: worked on bom. some changes. added license
Parts:
- C600, C601, R600, R601: JLC_placed_by (none) -> yes
- JP600, JP603, JP604, JP605: JLC_placed_by (none) -> never
- JP601, JP602: JLC_placed_by (none) -> no
- TP17: JLC_placed_by (none) -> never; now left out of the parts list
Changed lines of the file:
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@@
+      (effects (font (size 1.27 1.27)) hide)
+    )
+    (property "JLC_placed_by" "yes" (id 10) (at 175.26 68.58 0)
       (effects (font (size 1.27 1.27)) hide)
     )
@@
       (effects (font (size 1.27 1.27)) hide)
     )
+    (property "JLC_placed_by" "yes" (id 10) (at 99.06 67.31 0)
+      (effects (font (size 1.27 1.27)) hide)
+    )
     (pin "1")
     (pin "2")
@@
       (effects (font (size 1.27 1.27)) hide)
     )
+    (property "JLC_placed_by" "no" (id 5) (at 114.3 50.8 0)
+      (effects (font (size 1.27 1.27)) hide)
+    )
     (pin "1")
     (pin "2")
@@
   )
   (symbol (lib_id "Connector:TestPoint") (at 182.88 63.5 0) (unit 1)
-    (in_bom yes) (on_board yes)
+    (in_bom no) (on_board yes)
     (property "Reference" "TP17" (id 0) (at 184.2771 60.5091 0)
       (effects (font (size 1.27 1.27)) (justify left))
@@
     )
     (property "Supplier" "--" (id 4) (at 182.88 63.5 0)
+      (effects (font (size 1.27 1.27)) hide)
+    )
+    (property "JLC_placed_by" "never" (id 5) (at 182.88 63.5 0)
       (effects (font (size 1.27 1.27)) hide)
     )
@@
       (effects (font (size 1.27 1.27)) hide)
     )
+    (property "JLC_placed_by" "never" (id 5) (at 152.4 60.96 0)
+      (effects (font (size 1.27 1.27)) hide)
+    )
     (pin "1")
     (pin "2")
@@
     )
     (property "Supplier" "--" (id 4) (at 157.48 50.8 0)
+      (effects (font (size 1.27 1.27)) hide)
+    )
+    (property "JLC_placed_by" "no" (id 5) (at 157.48 50.8 0)
       (effects (font (size 1.27 1.27)) hide)
     )
@@
       (effects (font (size 1.27 1.27)) hide)
     )
+    (property "JLC_placed_by" "never" (id 5) (at 191.77 68.58 0)
+      (effects (font (size 1.27 1.27)) hide)
+    )
     (pin "1")
     (pin "2")
@@
       (effects (font (size 1.27 1.27)) hide)
     )
+    (property "JLC_placed_by" "never" (id 5) (at 116.84 60.96 0)
+      (effects (font (size 1.27 1.27)) hide)
+    )
     (pin "1")
     (pin "2")
@@
       (effects (font (size 1.27 1.27)) hide)
     )
+    (property "JLC_placed_by" "yes" (id 10) (at 182.88 76.2 0)
+      (effects (font (size 1.27 1.27)) hide)
+    )
     (pin "1")
     (pin "2")
@@
       (effects (font (size 1.27 1.27)) hide)
     )
+    (property "JLC_placed_by" "never" (id 5) (at 81.28 67.31 0)
+      (effects (font (size 1.27 1.27)) hide)
+    )
     (pin "1")
     (pin "2")
@@
       (effects (font (size 1.27 1.27)) hide)
     )
+    (property "JLC_placed_by" "yes" (id 10) (at 91.44 73.66 0)
+      (effects (font (size 1.27 1.27)) hide)
+    )
