File: raspberry.kicad_sch (KiCad schematic)
At the start: 7 parts

Commit message: Cleaned up board, replaced GPIO footprint with unshrouded version
Parts:
- JP400: footprint Connector_IDC:IDC-Header_2x20_P2.54mm_Vertical -> Connector_PinSocket_2.54mm:PinSocket_2x20_P2.54mm_Vertical
Connections:
- net +5V renamed 5V
- net VCC renamed 3V3
Changed lines of the file:
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@@
   (junction (at 147.32 129.54) (diameter 1.016) (color 0 0 0 0))
   (junction (at 149.86 129.54) (diameter 1.016) (color 0 0 0 0))
-  (junction (at 151.13 49.53) (diameter 1.016) (color 0 0 0 0))
+  (junction (at 152.4 49.53) (diameter 0) (color 0 0 0 0))
   (junction (at 152.4 129.54) (diameter 1.016) (color 0 0 0 0))
   (junction (at 153.67 129.54) (diameter 1.016) (color 0 0 0 0))
   (junction (at 154.94 129.54) (diameter 1.016) (color 0 0 0 0))
   (junction (at 157.48 129.54) (diameter 1.016) (color 0 0 0 0))
-  (junction (at 158.75 49.53) (diameter 1.016) (color 0 0 0 0))
+  (junction (at 160.02 49.53) (diameter 0) (color 0 0 0 0))
   (junction (at 160.02 129.54) (diameter 1.016) (color 0 0 0 0))
   (junction (at 198.12 76.2) (diameter 1.016) (color 0 0 0 0))
@@
     (stroke (width 0) (type solid) (color 0 0 0 0))
   )
-  (wire (pts (xy 143.51 31.75) (xy 143.51 35.56))
+  (wire (pts (xy 144.78 124.46) (xy 144.78 129.54))
+    (stroke (width 0) (type solid) (color 0 0 0 0))
+  )
+  (wire (pts (xy 144.78 129.54) (xy 147.32 129.54))
+    (stroke (width 0) (type solid) (color 0 0 0 0))
+  )
+  (wire (pts (xy 147.32 124.46) (xy 147.32 129.54))
+    (stroke (width 0) (type solid) (color 0 0 0 0))
+  )
+  (wire (pts (xy 147.32 129.54) (xy 149.86 129.54))
+    (stroke (width 0) (type solid) (color 0 0 0 0))
+  )
+  (wire (pts (xy 149.86 49.53) (xy 152.4 49.53))
+    (stroke (width 0) (type solid) (color 0 0 0 0))
+  )
+  (wire (pts (xy 149.86 58.42) (xy 149.86 49.53))
+    (stroke (width 0) (type solid) (color 0 0 0 0))
+  )
+  (wire (pts (xy 149.86 124.46) (xy 149.86 129.54))
+    (stroke (width 0) (type solid) (color 0 0 0 0))
+  )
+  (wire (pts (xy 149.86 129.54) (xy 152.4 129.54))
+    (stroke (width 0) (type solid) (color 0 0 0 0))
+  )
+  (wire (pts (xy 152.4 45.72) (xy 152.4 49.53))
     (stroke (width 0) (type default) (color 0 0 0 0))
   )
-  (wire (pts (xy 144.78 124.46) (xy 144.78 129.54))
-    (stroke (width 0) (type solid) (color 0 0 0 0))
-  )
-  (wire (pts (xy 144.78 129.54) (xy 147.32 129.54))
-    (stroke (width 0) (type solid) (color 0 0 0 0))
-  )
-  (wire (pts (xy 147.32 124.46) (xy 147.32 129.54))
-    (stroke (width 0) (type solid) (color 0 0 0 0))
-  )
-  (wire (pts (xy 147.32 129.54) (xy 149.86 129.54))
-    (stroke (width 0) (type solid) (color 0 0 0 0))
-  )
-  (wire (pts (xy 149.86 49.53) (xy 151.13 49.53))
-    (stroke (width 0) (type solid) (color 0 0 0 0))
-  )
-  (wire (pts (xy 149.86 58.42) (xy 149.86 49.53))
-    (stroke (width 0) (type solid) (color 0 0 0 0))
-  )
-  (wire (pts (xy 149.86 124.46) (xy 149.86 129.54))
-    (stroke (width 0) (type solid) (color 0 0 0 0))
-  )
-  (wire (pts (xy 149.86 129.54) (xy 152.4 129.54))
-    (stroke (width 0) (type solid) (color 0 0 0 0))
-  )
-  (wire (pts (xy 151.13 31.75) (xy 151.13 35.56))
+  (wire (pts (xy 152.4 58.42) (xy 152.4 49.53))
+    (stroke (width 0) (type solid) (color 0 0 0 0))
+  )
+  (wire (pts (xy 152.4 124.46) (xy 152.4 129.54))
+    (stroke (width 0) (type solid) (color 0 0 0 0))
+  )
+  (wire (pts (xy 152.4 129.54) (xy 153.67 129.54))
+    (stroke (width 0) (type solid) (color 0 0 0 0))
+  )
+  (wire (pts (xy 153.67 129.54) (xy 154.94 129.54))
+    (stroke (width 0) (type solid) (color 0 0 0 0))
+  )
+  (wire (pts (xy 154.94 124.46) (xy 154.94 129.54))
+    (stroke (width 0) (type solid) (color 0 0 0 0))
+  )
+  (wire (pts (xy 154.94 129.54) (xy 157.48 129.54))
+    (stroke (width 0) (type solid) (color 0 0 0 0))
+  )
+  (wire (pts (xy 157.48 49.53) (xy 160.02 49.53))
+    (stroke (width 0) (type solid) (color 0 0 0 0))
+  )
+  (wire (pts (xy 157.48 58.42) (xy 157.48 49.53))
+    (stroke (width 0) (type solid) (color 0 0 0 0))
+  )
+  (wire (pts (xy 157.48 124.46) (xy 157.48 129.54))
+    (stroke (width 0) (type solid) (color 0 0 0 0))
+  )
+  (wire (pts (xy 157.48 129.54) (xy 160.02 129.54))
+    (stroke (width 0) (type solid) (color 0 0 0 0))
+  )
+  (wire (pts (xy 160.02 45.72) (xy 160.02 49.53))
     (stroke (width 0) (type default) (color 0 0 0 0))
   )
-  (wire (pts (xy 151.13 49.53) (xy 152.4 49.53))
-    (stroke (width 0) (type solid) (color 0 0 0 0))
-  )
-  (wire (pts (xy 152.4 58.42) (xy 152.4 49.53))
-    (stroke (width 0) (type solid) (color 0 0 0 0))
-  )
-  (wire (pts (xy 152.4 124.46) (xy 152.4 129.54))
-    (stroke (width 0) (type solid) (color 0 0 0 0))
-  )
-  (wire (pts (xy 152.4 129.54) (xy 153.67 129.54))
-    (stroke (width 0) (type solid) (color 0 0 0 0))
-  )
-  (wire (pts (xy 153.67 129.54) (xy 154.94 129.54))
-    (stroke (width 0) (type solid) (color 0 0 0 0))
-  )
-  (wire (pts (xy 154.94 124.46) (xy 154.94 129.54))
-    (stroke (width 0) (type solid) (color 0 0 0 0))
-  )
-  (wire (pts (xy 154.94 129.54) (xy 157.48 129.54))
-    (stroke (width 0) (type solid) (color 0 0 0 0))
-  )
-  (wire (pts (xy 157.48 49.53) (xy 158.75 49.53))
-    (stroke (width 0) (type solid) (color 0 0 0 0))
-  )
-  (wire (pts (xy 157.48 58.42) (xy 157.48 49.53))
-    (stroke (width 0) (type solid) (color 0 0 0 0))
-  )
-  (wire (pts (xy 157.48 124.46) (xy 157.48 129.54))
-    (stroke (width 0) (type solid) (color 0 0 0 0))
-  )
-  (wire (pts (xy 157.48 129.54) (xy 160.02 129.54))
-    (stroke (width 0) (type solid) (color 0 0 0 0))
-  )
-  (wire (pts (xy 160.02 49.53) (xy 158.75 49.53))
-    (stroke (width 0) (type solid) (color 0 0 0 0))
+  (wire (pts (xy 160.02 49.53) (xy 203.2 49.53))
+    (stroke (width 0) (type default) (color 0 0 0 0))
   )
   (wire (pts (xy 160.02 58.42) (xy 160.02 49.53))
@@
     (effects (font (size 1.27 1.27)) (justify right))
   )
-  (hierarchical_label "+5V" (shape output) (at 143.51 35.56 270)
-    (effects (font (size 1.27 1.27)) (justify right))
-  )
-  (hierarchical_label "VCC" (shape output) (at 151.13 35.56 270)
-    (effects (font (size 1.27 1.27)) (justify right))
+  (hierarchical_label "5V" (shape output) (at 152.4 45.72 90)
+    (effects (font (size 1.27 1.27)) (justify left))
+  )
+  (hierarchical_label "3V3" (shape output) (at 160.02 45.72 90)
+    (effects (font (size 1.27 1.27)) (justify left))
   )
   (hierarchical_label "PREAMP1_EN" (shape output) (at 186.69 83.82 0)
@@
   (hierarchical_label "SCL" (shape bidirectional) (at 209.55 78.74 0)
     (effects (font (size 1.27 1.27)) (justify left))
-  )
-  (symbol (lib_id "power:+5V") (at 143.51 31.75 0) (unit 1)
-    (in_bom yes) (on_board yes)
-    (property "Reference" "#PWR0223" (id 0) (at 143.51 35.56 0)
-      (effects (font (size 1.27 1.27)) hide)
-    )
-    (property "Value" "+5V" (id 1) (at 143.8783 27.4256 0))
-    (property "Footprint" "" (id 2) (at 143.51 31.75 0)
-      (effects (font (size 1.27 1.27)) hide)
-    )
-    (property "Datasheet" "" (id 3) (at 143.51 31.75 0)
-      (effects (font (size 1.27 1.27)) hide)
-    )
-    (pin "1")
-  )
-  (symbol (lib_id "power:VCC") (at 151.13 31.75 0) (unit 1)
-    (in_bom yes) (on_board yes)
-    (property "Reference" "#PWR0224" (id 0) (at 151.13 35.56 0)
-      (effects (font (size 1.27 1.27)) hide)
-    )
-    (property "Value" "VCC" (id 1) (at 151.4983 27.4256 0))
-    (property "Footprint" "" (id 2) (at 151.13 31.75 0)
-      (effects (font (size 1.27 1.27)) hide)
-    )
-    (property "Datasheet" "" (id 3) (at 151.13 31.75 0)
-      (effects (font (size 1.27 1.27)) hide)
-    )
-    (pin "1")
-  )
-  (symbol (lib_id "power:+5V") (at 151.13 49.53 0) (unit 1)
-    (in_bom yes) (on_board yes)
-    (property "Reference" "#PWR0101" (id 0) (at 151.13 53.34 0)
-      (effects (font (size 1.27 1.27)) hide)
-    )
-    (property "Value" "+5V" (id 1) (at 151.4983 45.2056 0))
-    (property "Footprint" "" (id 2) (at 151.13 49.53 0)
-      (effects (font (size 1.27 1.27)) hide)
-    )
-    (property "Datasheet" "" (id 3) (at 151.13 49.53 0)
-      (effects (font (size 1.27 1.27)) hide)
-    )
-    (pin "1")
-  )
-  (symbol (lib_id "power:VCC") (at 158.75 49.53 0) (unit 1)
-    (in_bom yes) (on_board yes)
-    (property "Reference" "#PWR0102" (id 0) (at 158.75 53.34 0)
-      (effects (font (size 1.27 1.27)) hide)
-    )
-    (property "Value" "VCC" (id 1) (at 159.1183 45.2056 0))
-    (property "Footprint" "" (id 2) (at 158.75 49.53 0)
-      (effects (font (size 1.27 1.27)) hide)
-    )
-    (property "Datasheet" "" (id 3) (at 158.75 49.53 0)
-      (effects (font (size 1.27 1.27)) hide)
-    )
-    (pin "1")
-  )
-  (symbol (lib_id "power:VCC") (at 203.2 49.53 0) (unit 1)
-    (in_bom yes) (on_board yes)
-    (property "Reference" "#PWR0104" (id 0) (at 203.2 53.34 0)
-      (effects (font (size 1.27 1.27)) hide)
-    )
-    (property "Value" "VCC" (id 1) (at 203.5683 45.2056 0))
-    (property "Footprint" "" (id 2) (at 203.2 49.53 0)
-      (effects (font (size 1.27 1.27)) hide)
-    )
-    (property "Datasheet" "" (id 3) (at 203.2 49.53 0)
-      (effects (font (size 1.27 1.27)) hide)
-    )
-    (pin "1")
   )
   (symbol (lib_id "power:GND") (at 153.67 129.54 0) (unit 1)
@@
     (property "Reference" "JP400" (id 0) (at 165.1 56.4896 0))
     (property "Value" "Raspberry_Pi_2_3" (id 1) (at 170.18 58.7945 0))
-    (property "Footprint" "Connector_IDC:IDC-Header_2x20_P2.54mm_Vertical" (id 2) (at 154.94 91.44 0)
-      (effects (font (size 1.27 1.27)) hide)
-    )
+    (property "Footprint" "Connector_PinSocket_2.54mm:PinSocket_2x20_P2.54mm_Vertical" (id 2) (at 154.94 91.44 0)
+      (effects (font (size 1.27 1.27)) hide)
+    )

Commit message: Fixed references to library lost in transaction
Parts:
- JP400: footprint Connector_PinSocket_2.54mm:PinSocket_2x20_P2.54mm_Vertical -> muonpi-kicad-library:PinSocket_2x20_P2.54mm_Vertical; symbol Connector:Raspberry_Pi_2_3 -> muonpi-kicad-library:Raspberry_Pi_2_3
Changed lines of the file:
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@@
     (pin "2")
   )
-  (symbol (lib_id "Connector:Raspberry_Pi_2_3") (at 154.94 91.44 0) (unit 1)
+  (symbol (lib_id "muonpi-kicad-library:Raspberry_Pi_2_3") (at 154.94 91.44 0) (unit 1)
     (in_bom yes) (on_board yes)
     (property "Reference" "JP400" (id 0) (at 165.1 56.4896 0))
     (property "Value" "Raspberry_Pi_2_3" (id 1) (at 170.18 58.7945 0))
-    (property "Footprint" "Connector_PinSocket_2.54mm:PinSocket_2x20_P2.54mm_Vertical" (id 2) (at 154.94 91.44 0)
+    (property "Footprint" "muonpi-kicad-library:PinSocket_2x20_P2.54mm_Vertical" (id 2) (at 154.94 91.44 0)
       (effects (font (size 1.27 1.27)) hide)
     )
