File: raspberry.kicad_sch (KiCad schematic)
At the start: 7 parts

Commit message: worked on bom. some changes. added license
Parts:
- H1, H2, H3, H4: JLC_placed_by (none) -> never
- JP400: JLC_placed_by (none) -> no
- R410, R411: JLC_placed_by (none) -> yes
Changed lines of the file:
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@@
+      (effects (font (size 1.27 1.27)) hide)
+    )
+    (property "JLC_placed_by" "never" (id 5) (at 86.36 182.88 0)
       (effects (font (size 1.27 1.27)) hide)
     )
@@
       (effects (font (size 1.27 1.27)) hide)
     )
+    (property "JLC_placed_by" "never" (id 5) (at 86.36 177.8 0)
+      (effects (font (size 1.27 1.27)) hide)
+    )
   )
   (symbol (lib_id "Device:R") (at 198.12 68.58 0) (unit 1)
@@
     )
     (property "JLCplace" "C17673" (id 9) (at 198.12 68.58 0)
+      (effects (font (size 1.27 1.27)) hide)
+    )
+    (property "JLC_placed_by" "yes" (id 10) (at 198.12 68.58 0)
       (effects (font (size 1.27 1.27)) hide)
     )
@@
     )
     (property "Supplier" "LCSC" (id 7) (at 154.94 91.44 0)
+      (effects (font (size 1.27 1.27)) hide)
+    )
+    (property "JLC_placed_by" "no" (id 8) (at 154.94 91.44 0)
       (effects (font (size 1.27 1.27)) hide)
     )
@@
       (effects (font (size 1.27 1.27)) hide)
     )
+    (property "JLC_placed_by" "never" (id 5) (at 86.36 187.96 0)
+      (effects (font (size 1.27 1.27)) hide)
+    )
   )
   (symbol (lib_id "Device:R") (at 208.28 68.58 0) (unit 1)
@@
     )
     (property "JLCplace" "C17673" (id 9) (at 208.28 68.58 0)
+      (effects (font (size 1.27 1.27)) hide)
+    )
+    (property "JLC_placed_by" "yes" (id 10) (at 208.28 68.58 0)
       (effects (font (size 1.27 1.27)) hide)
     )
@@
       (effects (font (size 1.27 1.27)) hide)
     )
+    (property "JLC_placed_by" "never" (id 5) (at 86.36 172.72 0)
+      (effects (font (size 1.27 1.27)) hide)
+    )
